File: ThumbsUp.sch (KiCad schematic (older format))
At the start: 212 parts, among them IC1 RP2040, IC2 W25Q128JVSIM, IC3 RP2040, IC4 W25Q128JVSIM, J1 Conn_01x04_Male, J10 Raiser_Male, J11 Raiser_Female, J12 Raiser_Male, J13 Raiser_Female, J14 Raiser_Male, J15 Raiser_Female, J16 Raiser_Male, J17 Raiser_Female, J18 Raiser_Male, J19 Raiser_Female, J2 Conn_01x04_Male, J20 Conn_01x04_Female, J21 Conn_01x04_Female, J22 Conn_01x04_Female, J23 Conn_01x04_Female, J24 Conn_01x04_Male, J25 Conn_01x04_Male, J26 Conn_01x04_Male, J27 Conn_01x04_Male, J28 Conn_01x04_Female, J29 Conn_01x04_Female, J3 Conn_01x04_Female, J30 Conn_01x04_Female, J31 Conn_01x04_Female, J32 USB_C_Receptacle_USB2.0, J33 Raiser_Male, J34 Raiser_Female, J35 Raiser_Male, J36 PJ-3200B, J37 USB_C_Receptacle_USB2.0, J38 Raiser_Female, J39 Raiser_Male, J4 Conn_01x04_Male, J40 Raiser_Female, J41 Raiser_Male, J42 Raiser_Female, J43 Raiser_Male, J44 Raiser_Female, J45 Raiser_Male, J46 PJ-3200B, J47 Raiser_Female, J48 Raiser_Male, J49 Raiser_Female, J5 Conn_01x04_Female, J50 Raiser_Male, J51 Raiser_Female, J52 Raiser_Male, J53 Conn_01x04_Male, J54 Conn_01x04_Male, J55 Conn_01x04_Male, J56 Conn_01x04_Male, J57 Conn_01x04_Male, J58 Conn_01x04_Male, J59 Raiser_Male, J6 Conn_01x04_Male, J60 Raiser_Male, J61 Raiser_Male, J62 Raiser_Male, J63 Raiser_Male, J64 Raiser_Male, J65 Raiser_Male, J66 Raiser_Male, J67 Raiser_Male, J68 Raiser_Male, J69 Raiser_Male, J7 Conn_01x04_Male, J70 Raiser_Male, J71 Raiser_Male, J72 Raiser_Male, J73 Raiser_Male, J74 Raiser_Male, J75 Raiser_Male, J76 Raiser_Male, J8 Conn_01x04_Male, J9 Raiser_Female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

Commit message: Updated BOMs, Gerbers.
Parts:
- removed MX57: SwThL, keyswitches:MX-GLP2-HotSwap, symbol ThumbsUp-rescue:MX-NoLED-MX_Alps_Hybrid
- removed MX58: SwThR, keyswitches:MX-GLP2-HotSwap, symbol ThumbsUp-rescue:MX-NoLED-MX_Alps_Hybrid
Connections:
- no-connect marks 156 -> 158
Changed lines of the file:
@@
 Wire Wire Line
 	15550 1200 15850 1200
-$Comp
-L ThumbsUp-rescue:MX-NoLED-MX_Alps_Hybrid MX58
-U 1 1 64E86BAF
-P 10000 15450
-F 0 "MX58" H 10033 15673 60  0000 C CNN
-F 1 "SwThR" H 10033 15599 20  0000 C CNN
-F 2 "keyswitches:MX-GLP2-HotSwap" H 9375 15425 60  0001 C CNN
-F 3 "" H 9375 15425 60  0001 C CNN
-	1    10000 15450
-	-1   0    0    -1
-$EndComp
-$Comp
-L ThumbsUp-rescue:MX-NoLED-MX_Alps_Hybrid MX57
-U 1 1 64E85D21
-P 8400 15450
-F 0 "MX57" H 8433 15673 60  0000 C CNN
-F 1 "SwThL" H 8433 15599 20  0000 C CNN
-F 2 "keyswitches:MX-GLP2-HotSwap" H 7775 15425 60  0001 C CNN
-F 3 "" H 7775 15425 60  0001 C CNN
-	1    8400 15450
-	-1   0    0    -1
-$EndComp
 Wire Wire Line
 	8100 15650 8100 14900
@@
 $EndComp
 Wire Wire Line
-	8250 15400 8250 15050
-Wire Wire Line
 	8000 15650 8100 15650
 Wire Wire Line
 	7800 15450 7800 15050
-Wire Wire Line
-	7800 15050 8250 15050
 $Comp
 L Connector:Conn_01x04_Male J4
@@
 	0    -1   1    0
 $EndComp
-Connection ~ 7800 15050
 Connection ~ 7450 15050
 Wire Wire Line
 	7450 15050 7800 15050
-Wire Wire Line
-	7650 14900 7650 15800
-Wire Wire Line
-	7650 15800 8450 15800
-Wire Wire Line
-	8450 15800 8450 15600
-Wire Wire Line
-	9850 15400 9850 15000
-Wire Wire Line
-	9850 15000 10150 15000
-Connection ~ 10150 15000
-Wire Wire Line
-	10050 15600 9700 15600
-Wire Wire Line
-	9700 15600 9700 14900
-Wire Wire Line
-	9700 14900 10350 14900
 Text GLabel 10350 14350 1    50   Input ~ 0
 K_THR
@@
 Wire Wire Line
 	19800 7250 20150 7250
+NoConn ~ 7650 14900
+NoConn ~ 10350 14900
 $EndSCHEMATC
